Commit message: 更新chassis_DD-S.xacro的base_link座標系使其在輪子軸心的平面上

File: chassis_description/urdf/chassis_DD-S.xacro (robot description, xacro)
@@ -4,8 +4,8 @@
        Chassis geometry parameters
   ══════════════════════════════════════════════ -->
-  <xacro:property name="front_x"   value="0.27732"  />  <!-- wheelbase/2 front  (m) -->
-  <xacro:property name="rear_x"    value="-0.27268" />  <!-- wheelbase/2 rear   (m) -->
+  <xacro:property name="front_x"   value="0.275"    />  <!-- wheelbase/2 front  (m) -->
+  <xacro:property name="rear_x"    value="-0.275"   />  <!-- wheelbase/2 rear   (m) -->
   <xacro:property name="track_y"   value="0.31105"  />  <!-- half track width   (m) -->
-  <xacro:property name="wheel_z"   value="0.0765"   />  <!-- wheel axis height  (m) -->
+  <xacro:property name="wheel_z"   value="0"        />  <!-- wheel axis height  (m) -->
   <xacro:property name="wheel_radius" value="0.2032"  />  <!-- wheel radius, 16" diameter (m) -->
   <!-- Wheel inertia (ixx == izz for axisymmetric wheel) -->
@@ -43,5 +43,5 @@
         <origin xyz="0 0 0" rpy="0 0 0" />
         <geometry>
-          <mesh filename="package://chassis_description/meshes/DD-s/wheel_${name}_link.STL" />
+          <mesh filename="package://chassis_description/meshes/DD-S/wheel_${name}_link.STL" />
         </geometry>
         <material name="wheel_${name}_color">
@@ -52,5 +52,5 @@
         <origin xyz="0 0 0" rpy="0 0 0" />
         <geometry>
-          <mesh filename="package://chassis_description/meshes/DD-s/wheel_${name}_link.STL" />
+          <mesh filename="package://chassis_description/meshes/DD-S/wheel_${name}_link.STL" />
         </geometry>
       </collision>
@@ -77,5 +77,5 @@
   <link name="base_link">
     <inertial>
-      <origin xyz="0.0031731 -0.0002491 0.14649" rpy="0 0 0" />
+      <origin xyz="0.00084846 -0.0002491 0.06999" rpy="0 0 0" />
       <mass value="11.221" />
       <inertia
@@ -87,5 +87,5 @@
       <origin xyz="0 0 0" rpy="0 0 0" />
       <geometry>
-        <mesh filename="package://chassis_description/meshes/DD-s/base_link.STL" />
+        <mesh filename="package://chassis_description/meshes/DD-S/base_link.STL" />
       </geometry>
       <material name="white">
@@ -96,5 +96,5 @@
       <origin xyz="0 0 0" rpy="0 0 0" />
       <geometry>
-        <mesh filename="package://chassis_description/meshes/DD-s/base_link.STL" />
+        <mesh filename="package://chassis_description/meshes/DD-S/base_link.STL" />
       </geometry>
     </collision>
