Commit message: fix(all)
修改車體名稱從DD-S修改成DD-M

File: chassis_description/urdf/chassis_DD-M.xacro (robot description, xacro)
@@ -43,5 +43,5 @@
         <origin xyz="0 0 0" rpy="0 0 0" />
         <geometry>
-          <mesh filename="package://chassis_description/meshes/DD-S/wheel_${name}_link.STL" />
+          <mesh filename="package://chassis_description/meshes/DD-M/wheel_${name}_link.STL" />
         </geometry>
         <material name="wheel_${name}_color">
@@ -52,5 +52,5 @@
         <origin xyz="0 0 0" rpy="0 0 0" />
         <geometry>
-          <mesh filename="package://chassis_description/meshes/DD-S/wheel_${name}_link.STL" />
+          <mesh filename="package://chassis_description/meshes/DD-M/wheel_${name}_link.STL" />
         </geometry>
       </collision>
@@ -87,5 +87,5 @@
       <origin xyz="0 0 0" rpy="0 0 0" />
       <geometry>
-        <mesh filename="package://chassis_description/meshes/DD-S/base_link.STL" />
+        <mesh filename="package://chassis_description/meshes/DD-M/base_link.STL" />
       </geometry>
       <material name="white">
@@ -96,5 +96,5 @@
       <origin xyz="0 0 0" rpy="0 0 0" />
       <geometry>
-        <mesh filename="package://chassis_description/meshes/DD-S/base_link.STL" />
+        <mesh filename="package://chassis_description/meshes/DD-M/base_link.STL" />
       </geometry>
     </collision>
