Commit message: feat: Enhance chassis model support and add DD-M-HH variant
- Updated .gitignore to exclude additional local settings and protocol files.
- Modified README.md to include new chassis model DD-M-LH.
- Added vehicle parameters for the new DD-M-HH chassis model in vehicle_param_DD-M-HH.yaml.
- Enhanced bringup.launch.py to support dynamic model loading from models.yaml.
- Created model_registry.py to manage chassis model configurations.
- Added new meshes and URDF files for the DD-M-HH chassis model.
- Introduced chassis_common.xacro for shared components across chassis models.

File: chassis_description/urdf/chassis_DD-M-HH.xacro (robot description, xacro)
@@ -1,3 +1,16 @@
 <?xml version="1.0" encoding="utf-8"?>
+<!--
+  DD-M-HH — DD-M 的加高車身衍生型（噴藥車底盤）。
+  座標系說明（重要）：
+  SolidWorks 匯出的 DD-M-HH.SLDASM.urdf 其組合圖全域座標相對 DD-M **繞 Z 轉了 180°**
+  ——四個輪關節都帶 rpy="0 0 3.1416"，且 front_left 落在 x = -0.28。
+  本檔已把整車轉回 ROS 慣例（+x 為車頭、+y 為左側）：
+    p_ROS = Rz(pi) * p_SW
+  因此相對 SW 匯出值：
+    - 關節原點 x、y 取反號，關節 rpy 由 3.1416 變回 0（Rz(pi)*Rz(pi) = I）
+    - base_link 的 visual/collision 補上 rpy="0 0 ${pi}"，mesh 才會朝向正確
+    - base_link 慣性：質心 x、y 取反號，ixz／iyz 取反號（ixy 不變）
+    - 輪組 link 本身的座標系不變，故質量／慣性／com_y 與 SW 匯出值相同
+-->
 <robot name="chassis" xmlns:xacro="http://www.ros.org/wiki/xacro">
   <xacro:include filename="chassis_common.xacro" />
@@ -5,9 +18,9 @@
        Chassis geometry parameters
   ══════════════════════════════════════════════ -->
-  <xacro:property name="mesh_dir"  value="DD-M"     />  <!-- meshes/<mesh_dir>/ -->
-  <xacro:property name="front_x"   value="0.275"    />  <!-- wheelbase/2 front  (m) -->
-  <xacro:property name="rear_x"    value="-0.275"   />  <!-- wheelbase/2 rear   (m) -->
-  <xacro:property name="track_y"   value="0.31105"  />  <!-- half track width   (m) -->
-  <xacro:property name="wheel_z"   value="0"        />  <!-- wheel axis height  (m) -->
+  <xacro:property name="mesh_dir"  value="DD-M-HH"    />  <!-- meshes/<mesh_dir>/ -->
+  <xacro:property name="front_x"   value="0.28"       />  <!-- wheelbase/2 front  (m) -->
+  <xacro:property name="rear_x"    value="-0.28"      />  <!-- wheelbase/2 rear   (m) -->
+  <xacro:property name="track_y"   value="0.31105"    />  <!-- half track width   (m) -->
+  <xacro:property name="wheel_z"   value="-0.0056939" />  <!-- wheel axis height  (m) -->
   <xacro:property name="wheel_radius" value="0.2032"  />  <!-- wheel radius, 16" diameter (m) -->
   <!-- Wheel inertia (ixx == izz for axisymmetric wheel) -->
@@ -24,16 +37,17 @@
   <!-- ═══════════════════════════════════════════
        Base link
+       質心 Y 偏移 -0.12067 m 為 SolidWorks 匯出值（電池偏置），僅影響 Gazebo 動力學。
   ══════════════════════════════════════════════ -->
   <link name="base_link">
     <inertial>
-      <origin xyz="0.00084846 -0.0002491 0.06999" rpy="0 0 0" />
-      <mass value="11.221" />
+      <origin xyz="0.00017277 -0.12067 -0.00020488" rpy="0 0 0" />
+      <mass value="13.657" />
       <inertia
-        ixx="0.33572"  ixy="-3.5828E-09" ixz="-0.00054353"
-        iyy="0.54427"  iyz="-4.2841E-07"
-        izz="0.69255" />
+        ixx="0.54074"  ixy="2.1733E-06" ixz="1.9177E-08"
+        iyy="0.95687"  iyz="3.2487E-07"
+        izz="0.76507" />
     </inertial>
     <visual>
-      <origin xyz="0 0 0" rpy="0 0 0" />
+      <origin xyz="0 0 0" rpy="0 0 ${pi}" />
       <geometry>
         <mesh filename="package://chassis_description/meshes/${mesh_dir}/base_link.STL" />
@@ -44,5 +58,5 @@
     </visual>
     <collision>
-      <origin xyz="0 0 0" rpy="0 0 0" />
+      <origin xyz="0 0 0" rpy="0 0 ${pi}" />
       <geometry>
         <mesh filename="package://chassis_description/meshes/${mesh_dir}/base_link.STL" />
